Commit message: snoopy finally has collision working in the world ;)

File: snoopy/src/snoopy_description/description/config/snoopy_dimensions.xacro (robot description, xacro)
@@ -2,5 +2,7 @@
 <robot xmlns:xacro="http://www.ros.org/wiki/xacro">
   <xacro:property name="base_mass" value="0.334134" />
-  <xacro:property name="base_com_xyz" value="-0.018543979 0.00085988 0.03132396" />
+  <xacro:property name="base_com_x" value="-0.018543979" />
+  <xacro:property name="base_com_y" value="0.00085988" />
+  <xacro:property name="base_com_z" value="0.03132396" />
   <xacro:property name="base_ixx" value="0.00057643" />
   <xacro:property name="base_iyy" value="0.00361791" />
@@ -21,11 +23,19 @@
   <xacro:property name="joint_friction" value="0.0" />
   <xacro:property name="hip_mass" value="0.09551479" />
-  <xacro:property name="hip_com_xyz" value="0.036729 0.027408 0.001181" />
-  <xacro:property name="rh_hip_com_xyz" value="-0.036729 0.027408 0.001181" />
+  <xacro:property name="hip_com_x" value="0.036729" />
+  <xacro:property name="hip_com_y" value="0.027408" />
+  <xacro:property name="hip_com_z" value="0.001181" />
+  <xacro:property name="rh_hip_com_x" value="-0.036729" />
+  <xacro:property name="rh_hip_com_y" value="0.027408" />
+  <xacro:property name="rh_hip_com_z" value="0.001181" />
   <xacro:property name="hip_ixx" value="8.3668e-05" />
   <xacro:property name="hip_iyy" value="5.2898e-05" />
   <xacro:property name="hip_izz" value="0.00010700" />
   <xacro:property name="hip_mesh_LF" value="package://snoopy_description/meshes/LF_HIP.STL" />
-  <xacro:property name="thigh_mass_front" value="0.00708" /> <xacro:property name="thigh_mass_rear" value="0.00717" />  <xacro:property name="thigh_com_xyz" value="-0.04486 -0.00163 -0.02816" />
+  <xacro:property name="thigh_mass_front" value="0.00708" />
+  <xacro:property name="thigh_mass_rear" value="0.00717" />
+  <xacro:property name="thigh_com_x" value="-0.04486" />
+  <xacro:property name="thigh_com_y" value="-0.00163" />
+  <xacro:property name="thigh_com_z" value="-0.02816" />
   <xacro:property name="thigh_ixx" value="4.011e-06" />
   <xacro:property name="thigh_iyy" value="1.187e-05" />
@@ -35,6 +45,11 @@
   <xacro:property name="thigh_joint_offset_y" value="0.029523" />
   <xacro:property name="thigh_joint_offset_z" value="0.0012724" />
-  <xacro:property name="thigh_joint_rpy_base" value="0.436332" /> <xacro:property name="thigh_joint_rpy_mirror_r" value="-0.11522 0.436332 -0.1069" /> <xacro:property name="thigh_joint_rpy_mirror_l" value="0.11522 0.436332 0.1069" /> <xacro:property name="thigh_foot_mass" value="0.00294875" />
-  <xacro:property name="thigh_foot_com_xyz" value="0.04002 0.005801 -0.02456" />
+  <xacro:property name="thigh_joint_rpy_base" value="0.436332" />
+  <xacro:property name="thigh_joint_rpy_mirror_r" value="-0.11522 0.436332 -0.1069" />
+  <xacro:property name="thigh_joint_rpy_mirror_l" value="0.11522 0.436332 0.1069" />
+  <xacro:property name="thigh_foot_mass" value="0.00294875" />
+  <xacro:property name="thigh_foot_com_x" value="0.04002" />
+  <xacro:property name="thigh_foot_com_y" value="0.005801" />
+  <xacro:property name="thigh_foot_com_z" value="-0.02456" />
   <xacro:property name="thigh_foot_ixx" value="1.765e-06" />
   <xacro:property name="thigh_foot_iyy" value="6.375e-06" />
@@ -44,5 +59,7 @@
   <xacro:property name="foot_joint_offset_y" value="0.0023333" />
   <xacro:property name="foot_joint_offset_z" value="-0.12152" />
-  <xacro:property name="foot_joint_rpy_mirror_l" value="-3.1416 -2.35619 3.1416" /> <xacro:property name="foot_joint_rpy_mirror_r" value="3.1416 -2.35619 -3.1416" /> <xacro:property name="toe_mass" value="0.002" />
+  <xacro:property name="foot_joint_rpy_mirror_l" value="-3.1416 -2.35619 3.1416" />
+  <xacro:property name="foot_joint_rpy_mirror_r" value="3.1416 -2.35619 -3.1416" />
+  <xacro:property name="toe_mass" value="0.002" />
   <xacro:property name="toe_inertia" value="2e-08" />
   <xacro:property name="toe_radius" value="0.005" />

File: snoopy/src/snoopy_description/description/robot.urdf.xacro (robot description, xacro)
@@ -13,5 +13,5 @@
   <link name="base_link">
     <inertial>
-      <origin xyz="${base_com_xyz}" rpy="0 0 0" />
+      <origin xyz="${base_com_x} ${base_com_y} ${base_com_z}" rpy="0 0 0" />
       <mass value="${base_mass}" />
       <inertia

File: snoopy/src/snoopy_description/description/urdf/leg.urdf.xacro (robot description, xacro)
@@ -5,5 +5,5 @@
     <link name="${prefix}_HIP">
       <inertial>
-        <origin xyz="${hip_com_xyz}" rpy="0 0 0" />
+        <origin xyz="${hip_com_x} ${hip_com_y} ${hip_com_z}" rpy="0 0 0" />
         <mass value="${hip_mass}" />
         <inertia  ixx="${hip_ixx}" ixy="0" ixz="0" iyy="${hip_iyy}" iyz="0" izz="${hip_izz}" />
@@ -27,10 +27,12 @@
       <child link="${prefix}_HIP" />
       <dynamics damping="${joint_damping}" friction="${joint_friction}"/>
-      <axis xyz="1 0 0" /> <limit lower="${joint_lower_limit}" upper="${joint_upper_limit}" effort="${joint_effort_limit}" velocity="${joint_velocity_limit}" />
+      <axis xyz="1 0 0" />
+      <limit lower="${joint_lower_limit}" upper="${joint_upper_limit}" effort="${joint_effort_limit}" velocity="${joint_velocity_limit}" />
     </joint>
     <link name="${prefix}_THIGH">
       <inertial>
-        <origin xyz="${thigh_com_xyz}" rpy="0 0 0" />
-        <mass value="${thigh_mass_front}" /> <inertia ixx="${thigh_ixx}" ixy="0" ixz="0" iyy="${thigh_iyy}" iyz="0" izz="${thigh_izz}" />
+        <origin xyz="${thigh_com_x} ${thigh_com_y} ${thigh_com_z}" rpy="0 0 0" />
+        <mass value="${thigh_mass_front}" />
+        <inertia ixx="${thigh_ixx}" ixy="0" ixz="0" iyy="${thigh_iyy}" iyz="0" izz="${thigh_izz}" />
       </inertial>
       <visual>
@@ -40,4 +42,10 @@
         </geometry>
       </visual>
+      <collision>
+        <origin xyz="0 0 0" rpy="0 0 0" />
+        <geometry>
+          <mesh filename="package://snoopy_description/meshes/${thigh_mesh}" />
+        </geometry>
+      </collision>
     </link>
     <joint name="${prefix}_THIGH_JOINT" type="revolute">
@@ -47,9 +55,10 @@
       <child link="${prefix}_THIGH" />
       <dynamics damping="${joint_damping}" friction="${joint_friction}"/>
-      <axis xyz="0 1 0" /> <limit lower="${joint_lower_limit}" upper="${joint_upper_limit}" effort="${joint_effort_limit}" velocity="${joint_velocity_limit}" />
+      <axis xyz="0 1 0" />
+      <limit lower="${joint_lower_limit}" upper="${joint_upper_limit}" effort="${joint_effort_limit}" velocity="${joint_velocity_limit}" />
     </joint>
     <link name="${prefix}_THIGH_FOOT">
       <inertial>
-        <origin xyz="${thigh_foot_com_xyz}" rpy="0 0 0" />
+        <origin xyz="${thigh_foot_com_x} ${thigh_foot_com_y} ${thigh_foot_com_z}" rpy="0 0 0" />
         <mass value="${thigh_foot_mass}" />
         <inertia ixx="${thigh_foot_ixx}" ixy="0" ixz="0" iyy="${thigh_foot_iyy}" iyz="0" izz="${thigh_foot_izz}" />
@@ -74,5 +83,6 @@
       <child link="${prefix}_THIGH_FOOT" />
       <dynamics damping="${joint_damping}" friction="${joint_friction}"/>
-      <axis xyz="0 1 0" /> <limit lower="${joint_lower_limit}" upper="${joint_upper_limit}" effort="${joint_effort_limit}" velocity="${joint_velocity_limit}" />
+      <axis xyz="0 1 0" />
+      <limit lower="${joint_lower_limit}" upper="${joint_upper_limit}" effort="${joint_effort_limit}" velocity="${joint_velocity_limit}" />
     </joint>
     <link name="${prefix}_TOE">

Commit message: Added IK to the robot

File: snoopy/src/snoopy_description/description/config/snoopy_dimensions.xacro (robot description, xacro)
@@ -21,5 +21,5 @@
   <xacro:property name="joint_velocity_limit" value="2.5" />
   <xacro:property name="joint_damping" value="0.01" />
-  <xacro:property name="joint_friction" value="0.0" />
+  <xacro:property name="joint_friction" value="0.01" />
   <xacro:property name="hip_mass" value="0.09551479" />
   <xacro:property name="hip_com_x" value="0.036729" />
@@ -46,6 +46,8 @@
   <xacro:property name="thigh_joint_offset_z" value="0.0012724" />
   <xacro:property name="thigh_joint_rpy_base" value="0.436332" />
-  <xacro:property name="thigh_joint_rpy_mirror_r" value="-0.11522 0.436332 -0.1069" />
-  <xacro:property name="thigh_joint_rpy_mirror_l" value="0.11522 0.436332 0.1069" />
+  <!-- <xacro:property name="thigh_joint_rpy_mirror_r" value="-0.11522 0.436332 -0.1069" />
+  <xacro:property name="thigh_joint_rpy_mirror_l" value="0.11522 0.436332 0.1069" /> -->
+  <xacro:property name="thigh_joint_rpy_mirror_r" value="0 0 0" />
+  <xacro:property name="thigh_joint_rpy_mirror_l" value="0 0 0" />
   <xacro:property name="thigh_foot_mass" value="0.00294875" />
   <xacro:property name="thigh_foot_com_x" value="0.04002" />
@@ -59,6 +61,8 @@
   <xacro:property name="foot_joint_offset_y" value="0.0023333" />
   <xacro:property name="foot_joint_offset_z" value="-0.12152" />
-  <xacro:property name="foot_joint_rpy_mirror_l" value="-3.1416 -2.35619 3.1416" />
-  <xacro:property name="foot_joint_rpy_mirror_r" value="3.1416 -2.35619 -3.1416" />
+  <!-- <xacro:property name="foot_joint_rpy_mirror_l" value="-3.1416 -2.35619 3.1416" />
+  <xacro:property name="foot_joint_rpy_mirror_r" value="3.1416 -2.35619 -3.1416" /> -->
+  <xacro:property name="foot_joint_rpy_mirror_l" value="0 0 0" />
+  <xacro:property name="foot_joint_rpy_mirror_r" value="0 0 0" />
   <xacro:property name="toe_mass" value="0.002" />
   <xacro:property name="toe_inertia" value="2e-08" />

File: snoopy/src/snoopy_description/description/urdf/snoopy.ros2_control.xacro (robot description, xacro)
@@ -8,5 +8,5 @@
       <xacro:macro name="leg_ros2_control_joints" params="prefix">
         <joint name="${prefix}_HIP_JOINT">
-          <command_interface name="effort"/>
+          <command_interface name="position"/>
           <state_interface name="position">
             <param name="initial_value">0.0</param>
@@ -16,7 +16,7 @@
         </joint>
         <joint name="${prefix}_THIGH_JOINT">
-          <command_interface name="effort"/>
+          <command_interface name="position"/>
           <state_interface name="position">
-            <param name="initial_value">0.0</param>
+            <param name="initial_value">0.6</param>
           </state_interface>
           <state_interface name="velocity"/>
@@ -24,7 +24,7 @@
         </joint>
         <joint name="${prefix}_THIGH_FOOT_JOINT">
-          <command_interface name="effort"/>
+          <command_interface name="position"/>
           <state_interface name="position">
-            <param name="initial_value">0.0</param>
+            <param name="initial_value">-0.9</param>
           </state_interface>
           <state_interface name="velocity"/>

Commit message: Added velocity subscriber

File: snoopy/src/snoopy_description/description/config/snoopy_dimensions.xacro (robot description, xacro)
@@ -19,5 +19,5 @@
   <xacro:property name="joint_upper_limit" value="3.14" />
   <xacro:property name="joint_effort_limit" value="500" />
-  <xacro:property name="joint_velocity_limit" value="2.5" />
+  <xacro:property name="joint_velocity_limit" value="30" />
   <xacro:property name="joint_damping" value="0.01" />
   <xacro:property name="joint_friction" value="0.01" />

File: snoopy/src/snoopy_description/description/urdf/leg.urdf.xacro (robot description, xacro)
@@ -103,12 +103,4 @@
           <sphere radius="${toe_radius}"/>
         </geometry>
-        <surface>
-          <friction>
-            <ode>
-              <mu>0.3</mu>
-              <mu2>0.3</mu2>
-            </ode>
-          </friction>
-        </surface>
       </collision>
     </link>
@@ -120,8 +112,8 @@
     <gazebo reference="${prefix}_TOE">
         <kp>1000000.0</kp>
-        <kd>1.0</kd>
+        <kd>25.0</kd>
         <mu1>0.8</mu1>
         <mu2>0.8</mu2>
-        <maxVel>0.0</maxVel>
+        <maxVel>0.1</maxVel>
         <minDepth>0.001</minDepth>
     </gazebo>
