Commit message: Fixed issues with URDF. Added gait scheduler as a python package.

File: snoopy/src/snoopy_description/description/robot.urdf.xacro (robot description, xacro)
@@ -46,5 +46,5 @@
     thigh_mesh="LF_THIGH.STL"
     thigh_foot_mesh="LF_THIGH_FOOT.STL"
-    hip_visual_offset_rpy="0 0 0"
+    innertial_mirror="1"
   />
   <xacro:leg
@@ -59,5 +59,5 @@
     thigh_mesh="RF_THIGH.STL"
     thigh_foot_mesh="RF_THIGH_FOOT.STL"
-    hip_visual_offset_rpy="0 0 0"
+    innertial_mirror="-1"
   />
   <xacro:leg
@@ -72,5 +72,5 @@
     thigh_mesh="LH_THIGH.STL"
     thigh_foot_mesh="LH_THIGH_FOOT.STL"
-    hip_visual_offset_rpy="0 0 0"
+    innertial_mirror="1"
   />
   <xacro:leg
@@ -82,8 +82,8 @@
     thigh_joint_rpy="${thigh_joint_rpy_mirror_r}"
     foot_joint_rpy="${foot_joint_rpy_mirror_r}"
-    hip_mesh="LH_HIP.STL"
+    hip_mesh="RF_HIP.STL"
     thigh_mesh="RH_THIGH.STL"
     thigh_foot_mesh="RH_THIGH_FOOT.STL"
-    hip_visual_offset_rpy="3.14159 0 0"
+    innertial_mirror="-1"
   />
   <xacro:snoopy_ros2_control />

File: snoopy/src/snoopy_description/description/urdf/leg.urdf.xacro (robot description, xacro)
@@ -2,13 +2,13 @@
 <robot xmlns:xacro="http://www.ros.org/wiki/xacro">
   <xacro:include filename="$(find snoopy_description)/description/config/snoopy_dimensions.xacro" />
-  <xacro:macro name="leg" params="prefix parent_link hip_x hip_y hip_joint_rpy thigh_joint_rpy foot_joint_rpy hip_mesh thigh_mesh thigh_foot_mesh hip_visual_offset_rpy">
+  <xacro:macro name="leg" params="prefix parent_link hip_x hip_y hip_joint_rpy thigh_joint_rpy foot_joint_rpy hip_mesh thigh_mesh thigh_foot_mesh innertial_mirror">
     <link name="${prefix}_HIP">
       <inertial>
-        <origin xyz="${hip_com_x} ${hip_com_y} ${hip_com_z}" rpy="0 0 0" />
+        <origin xyz="${hip_com_x} ${hip_com_y * innertial_mirror} ${hip_com_z}" rpy="0 0 0" />
         <mass value="${hip_mass}" />
         <inertia  ixx="${hip_ixx}" ixy="0" ixz="0" iyy="${hip_iyy}" iyz="0" izz="${hip_izz}" />
       </inertial>
       <visual>
-        <origin xyz="0 0 0" rpy="${hip_visual_offset_rpy}" />
+        <origin xyz="0 0 0" rpy="0 0 0" />
         <geometry>
           <mesh filename="package://snoopy_description/meshes/${hip_mesh}" />
@@ -113,7 +113,7 @@
         <kp>1000000.0</kp>
         <kd>1.0</kd>
-        <mu1>0.8</mu1>
-        <mu2>0.8</mu2>
-        <maxVel>0.0</maxVel>
+        <mu1>100.0</mu1>
+        <mu2>100.0</mu2>
+        <maxVel>0.1</maxVel>
         <minDepth>0.001</minDepth>
     </gazebo>
